Commit message: feat: Inertia add and config to gazebo

File: urdf/mobile_base.xacro (robot description, xacro)
@@ -15,4 +15,11 @@
             <material name="blue" />
         </visual>
+        <collision>
+           <geometry>
+                <box size="${base_length} ${base_width} ${base_height}" />
+            </geometry>
+            <origin xyz="0 0 ${base_height / 2.0}" rpy="0 0 0" />
+            <material name="blue" />
+        </collision>
         <xacro:box_inertia m="5.0" l="${base_length}" w="${base_width}" h="${base_height}"
                            xyz="0 0 ${base_height / 2.0}" rpy="0 0 0" />
@@ -27,5 +34,11 @@
                 <material name="grey" />
             </visual>
-            <xacro:cylinder_inertia m="1.0" r="${wheel_radius}" h="${wheel_length}"
+            <collision>
+            <geometry>
+                    <cylinder radius="${wheel_radius}" length="${wheel_length}" />
+                </geometry>
+                <origin xyz="0 0 0" rpy="${pi / 2.0} 0 0" />
+            </collision>
+          <xacro:cylinder_inertia m="1.0" r="${wheel_radius}" h="${wheel_length}"
                                     xyz="0 0 0" rpy="${pi / 2.0} 0 0" />
         </link>
@@ -41,4 +54,10 @@
             <material name="grey" />
         </visual>
+        <collision>
+          <geometry>
+                <sphere radius="${wheel_radius / 2.0}" />
+            </geometry>
+            <origin xyz="0 0 0" rpy="0 0 0" />
+        </collision>
         <xacro:sphere_inertia m="0.5" r="${wheel_radius / 2.0}"
                               xyz="0 0 0" rpy="0 0 0" />
